File: prod/lattice_left.kicad_pcb (KiCad board)
At the start: 2 copper layers, 114.3 x 85.7 mm, 48 parts

Commit message: matrix finished
Parts:
- added J1: , USB_C_Receptacle, B.Cu at (95.2, 40.3)
- added J2: , USB_C_Receptacle, B.Cu at (190.5, 40.3)
- added U1: , RP2040, B.Cu at (152.4, 47.6)
- D1, D10, D11, D12, D13, D14, D15, D16, D17, D18, D19, D2, D20, D21, D22, D23, D24, D3, D4, D5, D6, D7, D8, D9: value 1N4148W -> (none); footprint lattice:D_SOD-123_via -> 1N4148W
- MX1, MX10, MX11, MX12, MX13, MX14, MX15, MX16, MX17, MX18, MX19, MX2, MX20, MX21, MX22, MX23, MX24, MX3, MX4, MX5, MX6, MX7, MX8, MX9: value MX_SW_HS -> (none); footprint marbastlib-mx:SW_MX_HS_1u -> MX_SW_HS
- moved D1 4.76 mm to (87.6, 114.3)
- moved D10 4.76 mm to (125.7, 95.2)
- moved D11 4.76 mm to (125.7, 76.2)
- moved D12 4.76 mm to (125.7, 57.2)
- moved D13 4.76 mm to (144.8, 114.3)
- moved D14 4.76 mm to (144.8, 95.2)
- moved D15 4.76 mm to (144.8, 76.2)
- moved D16 4.76 mm to (144.8, 57.2)
- moved D17 4.76 mm to (163.8, 114.3)
- moved D18 4.76 mm to (163.8, 95.2)
- moved D19 4.76 mm to (163.8, 76.2)
- moved D2 4.76 mm to (87.6, 95.2)
- moved D20 4.76 mm to (163.8, 57.2)
- moved D21 4.76 mm to (182.9, 114.3)
- moved D22 4.76 mm to (182.9, 95.2)
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Routing:
- net Net-(D1-K): track 95.2 -> 0.00 mm
Other:
- net class Default added: clearance 0.2, trace_width 0.25, via_dia 0.8, via_drill 0.4
