File: prod/lattice.kicad_pcb (KiCad board)
At the start: 2 copper layers, 114.3 x 85.7 mm, 71 parts

Commit message: trying ch552t version
Parts:
- removed C3, C4: , 22pF
- removed C5: , 100nF
- removed R3, R6, R7: , 1k
- removed R4, R5: , 27R
- removed SW1, SW2: , SW_Push
- removed U4: , XC6206PxxxMR
- removed Y1: , 12MHz
- U3: footprint RP2040 -> CH552T
- turned MX1 to 180 degrees
- turned MX10 to 180 degrees
- turned MX11 to 180 degrees
- turned MX12 to 180 degrees
- turned MX13 to 180 degrees
- turned MX14 to 180 degrees
- turned MX15 to 180 degrees
- turned MX16 to 180 degrees
- turned MX17 to 180 degrees
- turned MX18 to 180 degrees
- turned MX19 to 180 degrees
- turned MX2 to 180 degrees
- turned MX20 to 180 degrees
- turned MX21 to 180 degrees
- turned MX22 to 180 degrees
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Changed lines of the file:
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@@
   (page A4)
   (title_block
-    (title lattice_left)
-    (rev 2024.02)
+    (title lattice)
+    (rev 2024.03)
     (company sboysel)
   )
@@
   )
         (module MX_SW_HS (layer B.Cu)
-            (at 95.25 114.3 0)
+            (at 95.25 114.3 180)
             (fp_text reference "MX1" (at 0 0 0) (layer "B.Fab")
               (effects (font (size 1 1) (thickness 0.15)))
@@
         )
         (module MX_SW_HS (layer B.Cu)
-            (at 95.25 95.25 0)
+            (at 95.25 95.25 180)
             (fp_text reference "MX2" (at 0 0 0) (layer "B.Fab")
               (effects (font (size 1 1) (thickness 0.15)))
@@
         )
         (module MX_SW_HS (layer B.Cu)
-            (at 95.25 76.2 0)
+            (at 95.25 76.2 180)
             (fp_text reference "MX3" (at 0 0 0) (layer "B.Fab")
               (effects (font (size 1 1) (thickness 0.15)))
@@
         )
         (module MX_SW_HS (layer B.Cu)
-            (at 95.25 57.150000000000006 0)
+            (at 95.25 57.150000000000006 180)
             (fp_text reference "MX4" (at 0 0 0) (layer "B.Fab")
               (effects (font (size 1 1) (thickness 0.15)))
@@
         )
         (module MX_SW_HS (layer B.Cu)
-            (at 114.3 114.3 0)
+            (at 114.3 114.3 180)
             (fp_text reference "MX5" (at 0 0 0) (layer "B.Fab")
               (effects (font (size 1 1) (thickness 0.15)))
@@
         )
         (module MX_SW_HS (layer B.Cu)
-            (at 114.3 95.25 0)
+            (at 114.3 95.25 180)
             (fp_text reference "MX6" (at 0 0 0) (layer "B.Fab")
               (effects (font (size 1 1) (thickness 0.15)))
@@
         )
         (module MX_SW_HS (layer B.Cu)
-            (at 114.3 76.2 0)
+            (at 114.3 76.2 180)
             (fp_text reference "MX7" (at 0 0 0) (layer "B.Fab")
               (effects (font (size 1 1) (thickness 0.15)))
@@
         )
         (module MX_SW_HS (layer B.Cu)
-            (at 114.3 57.150000000000006 0)
+            (at 114.3 57.150000000000006 180)
             (fp_text reference "MX8" (at 0 0 0) (layer "B.Fab")
               (effects (font (size 1 1) (thickness 0.15)))
@@
         )
         (module MX_SW_HS (layer B.Cu)
-            (at 133.35 114.3 0)
+            (at 133.35 114.3 180)
             (fp_text reference "MX9" (at 0 0 0) (layer "B.Fab")
               (effects (font (size 1 1) (thickness 0.15)))
@@
         )
         (module MX_SW_HS (layer B.Cu)
-            (at 133.35 95.25 0)
+            (at 133.35 95.25 180)
             (fp_text reference "MX10" (at 0 0 0) (layer "B.Fab")
               (effects (font (size 1 1) (thickness 0.15)))
@@
         )
         (module MX_SW_HS (layer B.Cu)
-            (at 133.35 76.2 0)
+            (at 133.35 76.2 180)
             (fp_text reference "MX11" (at 0 0 0) (layer "B.Fab")
               (effects (font (size 1 1) (thickness 0.15)))
@@
         )
         (module MX_SW_HS (layer B.Cu)
-            (at 133.35 57.150000000000006 0)
+            (at 133.35 57.150000000000006 180)
             (fp_text reference "MX12" (at 0 0 0) (layer "B.Fab")
               (effects (font (size 1 1) (thickness 0.15)))
@@
         )
         (module MX_SW_HS (layer B.Cu)
-            (at 152.4 114.3 0)
+            (at 152.4 114.3 180)
             (fp_text reference "MX13" (at 0 0 0) (layer "B.Fab")
               (effects (font (size 1 1) (thickness 0.15)))
@@
         )
         (module MX_SW_HS (layer B.Cu)
-            (at 152.4 95.25 0)
+            (at 152.4 95.25 180)
             (fp_text reference "MX14" (at 0 0 0) (layer "B.Fab")
               (effects (font (size 1 1) (thickness 0.15)))
@@
         )
         (module MX_SW_HS (layer B.Cu)
-            (at 152.4 76.2 0)
+            (at 152.4 76.2 180)
             (fp_text reference "MX15" (at 0 0 0) (layer "B.Fab")
               (effects (font (size 1 1) (thickness 0.15)))
@@
         )
         (module MX_SW_HS (layer B.Cu)
-            (at 152.4 57.150000000000006 0)
+            (at 152.4 57.150000000000006 180)
             (fp_text reference "MX16" (at 0 0 0) (layer "B.Fab")
               (effects (font (size 1 1) (thickness 0.15)))
@@
         )
         (module MX_SW_HS (layer B.Cu)
-            (at 171.45 114.3 0)
+            (at 171.45 114.3 180)
             (fp_text reference "MX17" (at 0 0 0) (layer "B.Fab")
               (effects (font (size 1 1) (thickness 0.15)))
@@
         )
         (module MX_SW_HS (layer B.Cu)
-            (at 171.45 95.25 0)
+            (at 171.45 95.25 180)
             (fp_text reference "MX18" (at 0 0 0) (layer "B.Fab")
               (effects (font (size 1 1) (thickness 0.15)))
@@
         )
         (module MX_SW_HS (layer B.Cu)
-            (at 171.45 76.2 0)
+            (at 171.45 76.2 180)
             (fp_text reference "MX19" (at 0 0 0) (layer "B.Fab")
               (effects (font (size 1 1) (thickness 0.15)))
@@
         )
         (module MX_SW_HS (layer B.Cu)
-            (at 171.45 57.150000000000006 0)
+            (at 171.45 57.150000000000006 180)
             (fp_text reference "MX20" (at 0 0 0) (layer "B.Fab")
               (effects (font (size 1 1) (thickness 0.15)))
@@
         )
         (module MX_SW_HS (layer B.Cu)
-            (at 190.5 114.3 0)
+            (at 190.5 114.3 180)
             (fp_text reference "MX21" (at 0 0 0) (layer "B.Fab")
               (effects (font (size 1 1) (thickness 0.15)))
@@
         )
         (module MX_SW_HS (layer B.Cu)
-            (at 190.5 95.25 0)
+            (at 190.5 95.25 180)
             (fp_text reference "MX22" (at 0 0 0) (layer "B.Fab")
               (effects (font (size 1 1) (thickness 0.15)))
@@
         )
         (module MX_SW_HS (layer B.Cu)
-            (at 190.5 76.2 0)
+            (at 190.5 76.2 180)
             (fp_text reference "MX23" (at 0 0 0) (layer "B.Fab")
               (effects (font (size 1 1) (thickness 0.15)))
@@
         )
         (module MX_SW_HS (layer B.Cu)
-            (at 190.5 57.150000000000006 0)
+            (at 190.5 57.150000000000006 180)
             (fp_text reference "MX24" (at 0 0 0) (layer "B.Fab")
               (effects (font (size 1 1) (thickness 0.15)))
@@
             )
         )
-        (module 12MHz (layer B.Cu)
-            (at 123.82499999999999 42.862500000000004 0)
-            (fp_text reference "Y1" (at 0 0 0) (layer "B.Fab")
-              (effects (font (size 1 1) (thickness 0.15)))
-            )
-        )
-        (module 1k (layer B.Cu)
-            (at 124.82499999999999 47.62500000000001 90)
-            (fp_text reference "R3" (at 0 0 0) (layer "B.Fab")
-              (effects (font (size 1 1) (thickness 0.15)))
-            )
-        )
-        (module 22pF (layer B.Cu)
-            (at 123.82499999999999 47.62500000000001 90)
-            (fp_text reference "C3" (at 0 0 0) (layer "B.Fab")
-              (effects (font (size 1 1) (thickness 0.15)))
-            )
-        )
-        (module 22pF (layer B.Cu)
-            (at 122.82499999999999 47.62500000000001 90)
-            (fp_text reference "C4" (at 0 0 0) (layer "B.Fab")
-              (effects (font (size 1 1) (thickness 0.15)))
-            )
-        )
-        (module RP2040 (layer B.Cu)
+        (module CH552T (layer B.Cu)
             (at 133.35 43.62500000000001 90)
             (fp_text reference "U3" (at 0 0 0) (layer "B.Fab")
               (effects (font (size 1 1) (thickness 0.15)))
             )
-        )
-        (module 27R (layer B.Cu)
-            (at 142.875 41.862500000000004 0)
-            (fp_text reference "R4" (at 0 0 0) (layer "B.Fab")
-              (effects (font (size 1 1) (thickness 0.15)))
-            )
-        )
-        (module 27R (layer B.Cu)
-            (at 142.875 42.862500000000004 0)
-            (fp_text reference "R5" (at 0 0 0) (layer "B.Fab")
-              (effects (font (size 1 1) (thickness 0.15)))
-            )
-        )
-        (module 1k (layer B.Cu)
-            (at 142.875 43.862500000000004 0)
-            (fp_text reference "R6" (at 0 0 0) (layer "B.Fab")
-              (effects (font (size 1 1) (thickness 0.15)))
-            )
-        )
-        (module XC6206PxxxMR (layer B.Cu)
-            (at 152.4 43.862500000000004 270)
-            (fp_text reference "U4" (at 0 0 0) (layer "B.Fab")
-              (effects (font (size 1 1) (thickness 0.15)))
-            )
-        )
-        (module 1k (layer B.Cu)
-            (at 147.4 47.62500000000001 90)
-            (fp_text reference "R7" (at 0 0 0) (layer "B.Fab")
-              (effects (font (size 1 1) (thickness 0.15)))
-            )
-        )
-        (module 100nF (layer B.Cu)
-            (at 148.4 47.62500000000001 90)
-            (fp_text reference "C5" (at 0 0 0) (layer "B.Fab")
-              (effects (font (size 1 1) (thickness 0.15)))
-            )
-        )
-        (module SW_Push (layer B.Cu)
-            (at 95.25 68.2 0)
-            (fp_text reference "SW1" (at 0 0 0) (layer "B.Fab")
-              (effects (font (size 1 1) (thickness 0.15)))
-            )
-        )
-        (module SW_Push (layer B.Cu)
-            (at 114.3 68.2 0)
-            (fp_text reference "SW2" (at 0 0 0) (layer "B.Fab")
-              (effects (font (size 1 1) (thickness 0.15)))
-            )
