File: ergogen/output/pcbs/lattice_left.kicad_pcb (KiCad board)
At the start: 2 copper layers, 114.3 x 85.7 mm, 68 parts

Commit message: components placed
Parts:
- added C10: , 100nF, B.Cu at (133.8, 47.6)
- added C11: , 100nF, B.Cu at (135.8, 47.6)
- added C12: , 100nF, B.Cu at (137.8, 47.6)
- added C13: , 100nF, B.Cu at (139.8, 47.6)
- added C14: , 100nF, B.Cu at (141.8, 47.6)
- added C15: , 1uF, B.Cu at (119.1, 47.6)
- added C16: , 100nF, B.Cu at (121.1, 47.6)
- added C17: , 100nF, B.Cu at (123.1, 47.6)
- added C6: , 10uF, B.Cu at (125.8, 47.6)
- added C7: , 1uF, B.Cu at (127.8, 47.6)
- added C8: , 100nF, B.Cu at (129.8, 47.6)
- added C9: , 100nF, B.Cu at (131.8, 47.6)
- added R5: , 1k, B.Cu at (160.4, 44.9)
- added R6: , 1k, B.Cu at (166.7, 47.6)
- added R7: , 1k, B.Cu at (176.2, 47.6)
- R3, R4: footprint 1k -> 27R
- moved R4 16.5 mm to (160.4, 42.9)
- moved R3 9.23 mm to (160.4, 40.9)
- moved SW1 5.76 mm to (128.6, 41.9), turned to 0 degrees
- moved SW2 5.76 mm to (138.1, 41.9), turned to 0 degrees
- moved U4 1.59 mm to (168.3, 42.9)
- moved C4 1.00 mm to (181.0, 42.9)
- moved C5 1.00 mm to (181.0, 42.9)
Changed lines of the file:
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@@
+            )
+        )
+        (module 27R (layer B.Cu)
+            (at 160.4 40.862500000000004 0)
+            (fp_text reference "R3" (at 0 0 0) (layer "B.Fab")
+              (effects (font (size 1 1) (thickness 0.15)))
+            )
+        )
+        (module 27R (layer B.Cu)
+            (at 160.4 42.862500000000004 0)
+            (fp_text reference "R4" (at 0 0 0) (layer "B.Fab")
+              (effects (font (size 1 1) (thickness 0.15)))
+            )
+        )
+        (module 1k (layer B.Cu)
+            (at 160.4 44.862500000000004 0)
+            (fp_text reference "R5" (at 0 0 0) (layer "B.Fab")
+              (effects (font (size 1 1) (thickness 0.15)))
             )
         )
@@
         )
         (module XC6206PxxxMR (layer B.Cu)
-            (at 166.6875 42.862500000000004 0)
+            (at 168.27499999999998 42.862500000000004 0)
             (fp_text reference "U4" (at 0 0 0) (layer "B.Fab")
               (effects (font (size 1 1) (thickness 0.15)))
@@
         (module 1k (layer B.Cu)
             (at 166.6875 47.62500000000001 0)
-            (fp_text reference "R3" (at 0 0 0) (layer "B.Fab")
+            (fp_text reference "R6" (at 0 0 0) (layer "B.Fab")
               (effects (font (size 1 1) (thickness 0.15)))
             )
@@
         )
         (module 22pF (layer B.Cu)
-            (at 179.975 42.862500000000004 90)
+            (at 180.975 42.862500000000004 90)
             (fp_text reference "C4" (at 0 0 0) (layer "B.Fab")
               (effects (font (size 1 1) (thickness 0.15)))
@@
         )
         (module 22pF (layer B.Cu)
-            (at 181.975 42.862500000000004 90)
+            (at 180.975 42.862500000000004 90)
             (fp_text reference "C5" (at 0 0 0) (layer "B.Fab")
               (effects (font (size 1 1) (thickness 0.15)))
@@
         (module 1k (layer B.Cu)
             (at 176.21249999999998 47.62500000000001 0)
-            (fp_text reference "R4" (at 0 0 0) (layer "B.Fab")
+            (fp_text reference "R7" (at 0 0 0) (layer "B.Fab")
               (effects (font (size 1 1) (thickness 0.15)))
             )
         )
         (module SW_Push (layer B.Cu)
-            (at 128.5875 47.62500000000001 90)
+            (at 128.5875 41.862500000000004 0)
             (fp_text reference "SW1" (at 0 0 0) (layer "B.Fab")
               (effects (font (size 1 1) (thickness 0.15)))
@@
         )
         (module SW_Push (layer B.Cu)
-            (at 138.11249999999998 47.62500000000001 90)
+            (at 138.11249999999998 41.862500000000004 0)
             (fp_text reference "SW2" (at 0 0 0) (layer "B.Fab")
               (effects (font (size 1 1) (thickness 0.15)))
             )
+        )
+        (module 10uF (layer B.Cu)
+            (at 125.82499999999999 47.62500000000001 90)
+            (fp_text reference "C6" (at 0 0 0) (layer "B.Fab")
+              (effects (font (size 1 1) (thickness 0.15)))
+            )
+        )
+        (module 1uF (layer B.Cu)
+            (at 127.82499999999999 47.62500000000001 90)
+            (fp_text reference "C7" (at 0 0 0) (layer "B.Fab")
+              (effects (font (size 1 1) (thickness 0.15)))
+            )
+        )
+        (module 100nF (layer B.Cu)
+            (at 129.825 47.62500000000001 90)
+            (fp_text reference "C8" (at 0 0 0) (layer "B.Fab")
+              (effects (font (size 1 1) (thickness 0.15)))
+            )
+        )
+        (module 100nF (layer B.Cu)
+            (at 131.825 47.62500000000001 90)
+            (fp_text reference "C9" (at 0 0 0) (layer "B.Fab")
+              (effects (font (size 1 1) (thickness 0.15)))
+            )
+        )
+        (module 100nF (layer B.Cu)
+            (at 133.825 47.62500000000001 90)
+            (fp_text reference "C10" (at 0 0 0) (layer "B.Fab")
+              (effects (font (size 1 1) (thickness 0.15)))
+            )
+        )
+        (module 100nF (layer B.Cu)
+            (at 135.825 47.62500000000001 90)
+            (fp_text reference "C11" (at 0 0 0) (layer "B.Fab")
+              (effects (font (size 1 1) (thickness 0.15)))
+            )
+        )
+        (module 100nF (layer B.Cu)
+            (at 137.825 47.62500000000001 90)
+            (fp_text reference "C12" (at 0 0 0) (layer "B.Fab")
+              (effects (font (size 1 1) (thickness 0.15)))
+            )
+        )
+        (module 100nF (layer B.Cu)
+            (at 139.825 47.62500000000001 90)
+            (fp_text reference "C13" (at 0 0 0) (layer "B.Fab")
+              (effects (font (size 1 1) (thickness 0.15)))
+            )
+        )
+        (module 100nF (layer B.Cu)
+            (at 141.825 47.62500000000001 90)
+            (fp_text reference "C14" (at 0 0 0) (layer "B.Fab")
+              (effects (font (size 1 1) (thickness 0.15)))
+            )
+        )
+        (module 1uF (layer B.Cu)
+            (at 119.0625 47.62500000000001 90)
+            (fp_text reference "C15" (at 0 0 0) (layer "B.Fab")
+              (effects (font (size 1 1) (thickness 0.15)))
+            )
+        )
+        (module 100nF (layer B.Cu)
+            (at 121.0625 47.62500000000001 90)
+            (fp_text reference "C16" (at 0 0 0) (layer "B.Fab")
+              (effects (font (size 1 1) (thickness 0.15)))
+            )
+        )
+        (module 100nF (layer B.Cu)
+            (at 123.0625 47.62500000000001 90)
+            (fp_text reference "C17" (at 0 0 0) (layer "B.Fab")
+              (effects (font (size 1 1) (thickness 0.15)))
+            )

Commit message: adding breakout header
Parts:
- added J3: , Conn_01x05, B.Cu at (119.3, 66.7)
- moved C15 24.3 mm to (142.9, 52.4)
- moved C16 20.4 mm to (140.9, 52.4)
- moved C6 17.1 mm to (142.9, 47.6)
- moved C17 16.5 mm to (138.9, 52.4)
- moved C7 13.1 mm to (140.9, 47.6)
- moved C14 10.1 mm to (132.9, 52.4)
- moved C8 9.05 mm to (138.9, 47.6)
- moved C13 6.87 mm to (134.9, 52.4)
- moved C9 5.05 mm to (136.9, 47.6)
- moved C12 4.86 mm to (136.9, 52.4)
- moved C11 2.95 mm to (132.9, 47.6)
- moved C10 1.05 mm to (134.9, 47.6)
Changed lines of the file:
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@@
+            )
+        )
+        (module Conn_01x05 (layer B.Cu)
+            (at 119.3 66.675 90)
+            (fp_text reference "J3" (at 0 0 0) (layer "B.Fab")
+              (effects (font (size 1 1) (thickness 0.15)))
             )
         )
         (module 10uF (layer B.Cu)
-            (at 125.82499999999999 47.62500000000001 90)
+            (at 142.875 47.62500000000001 90)
             (fp_text reference "C6" (at 0 0 0) (layer "B.Fab")
               (effects (font (size 1 1) (thickness 0.15)))
@@
         )
         (module 1uF (layer B.Cu)
-            (at 127.82499999999999 47.62500000000001 90)
+            (at 140.875 47.62500000000001 90)
             (fp_text reference "C7" (at 0 0 0) (layer "B.Fab")
               (effects (font (size 1 1) (thickness 0.15)))
@@
         )
         (module 100nF (layer B.Cu)
-            (at 129.825 47.62500000000001 90)
+            (at 138.875 47.62500000000001 90)
             (fp_text reference "C8" (at 0 0 0) (layer "B.Fab")
               (effects (font (size 1 1) (thickness 0.15)))
@@
         )
         (module 100nF (layer B.Cu)
-            (at 131.825 47.62500000000001 90)
+            (at 136.875 47.62500000000001 90)
             (fp_text reference "C9" (at 0 0 0) (layer "B.Fab")
               (effects (font (size 1 1) (thickness 0.15)))
@@
         )
         (module 100nF (layer B.Cu)
-            (at 133.825 47.62500000000001 90)
+            (at 134.875 47.62500000000001 90)
             (fp_text reference "C10" (at 0 0 0) (layer "B.Fab")
               (effects (font (size 1 1) (thickness 0.15)))
@@
         )
         (module 100nF (layer B.Cu)
-            (at 135.825 47.62500000000001 90)
+            (at 132.875 47.62500000000001 90)
             (fp_text reference "C11" (at 0 0 0) (layer "B.Fab")
               (effects (font (size 1 1) (thickness 0.15)))
@@
         )
         (module 100nF (layer B.Cu)
-            (at 137.825 47.62500000000001 90)
+            (at 136.875 52.3875 90)
             (fp_text reference "C12" (at 0 0 0) (layer "B.Fab")
               (effects (font (size 1 1) (thickness 0.15)))
@@
         )
         (module 100nF (layer B.Cu)
-            (at 139.825 47.62500000000001 90)
+            (at 134.875 52.3875 90)
             (fp_text reference "C13" (at 0 0 0) (layer "B.Fab")
               (effects (font (size 1 1) (thickness 0.15)))
@@
         )
         (module 100nF (layer B.Cu)
-            (at 141.825 47.62500000000001 90)
+            (at 132.875 52.3875 90)
             (fp_text reference "C14" (at 0 0 0) (layer "B.Fab")
               (effects (font (size 1 1) (thickness 0.15)))
@@
         )
         (module 1uF (layer B.Cu)
-            (at 119.0625 47.62500000000001 90)
+            (at 142.875 52.3875 90)
             (fp_text reference "C15" (at 0 0 0) (layer "B.Fab")
               (effects (font (size 1 1) (thickness 0.15)))
@@
         )
         (module 100nF (layer B.Cu)
-            (at 121.0625 47.62500000000001 90)
+            (at 140.875 52.3875 90)
             (fp_text reference "C16" (at 0 0 0) (layer "B.Fab")
               (effects (font (size 1 1) (thickness 0.15)))
@@
         )
         (module 100nF (layer B.Cu)
-            (at 123.0625 47.62500000000001 90)
+            (at 138.875 52.3875 90)
             (fp_text reference "C17" (at 0 0 0) (layer "B.Fab")
               (effects (font (size 1 1) (thickness 0.15)))
@@
             )
             (gr_text "left" (at 104.775 104.77499999999999 0) (layer B.SilkS knockout)
-                (effects (font  (face "JetBrainsMono NF") (size 1 1) (thickness 0.15)) (justify mirror))
+                (effects (font (size 1 1) (thickness 0.15)) (justify mirror))
             )
             (gr_text "lattice v2024.02" (at 180.975 104.77499999999999 0) (layer B.SilkS knockout)
-                (effects (font  (face "JetBrainsMono NF") (size 1 1) (thickness 0.15)) (justify mirror))
+                (effects (font (size 1 1) (thickness 0.15)) (justify mirror))
             )
   (gr_line (start 85.725 120.825) (end 85.725 41.10000000000001) (angle 90) (layer Edge.Cuts) (width 0.15))

Commit message: placement adjustments
Parts:
- moved C1 11.7 mm to (104.8, 42.9), turned to 270 degrees
- moved U3 10.8 mm to (119.1, 42.9), turned to 270 degrees
- moved C10 4.53 mm to (130.3, 47.6)
- moved C11 4.53 mm to (128.3, 47.6)
- moved C12 4.53 mm to (132.3, 52.4)
- moved C13 4.53 mm to (130.3, 52.4)
- moved C14 4.53 mm to (128.3, 52.4)
- moved C15 4.53 mm to (138.3, 52.4)
- moved C16 4.53 mm to (136.3, 52.4)
- moved C17 4.53 mm to (134.3, 52.4)
- moved C6 4.53 mm to (138.3, 47.6)
- moved C7 4.53 mm to (136.3, 47.6)
- moved C8 4.53 mm to (134.3, 47.6)
- moved C9 4.53 mm to (132.3, 47.6)
- moved C2 4.17 mm to (114.3, 42.9), turned to 270 degrees
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Changed lines of the file:
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@@
         )
         (module RP2040 (layer B.Cu)
-            (at 152.4 45.243750000000006 45)
+            (at 152.4 45.243750000000006 225)
             (fp_text reference "U1" (at 0 0 0) (layer "B.Fab")
               (effects (font (size 1 1) (thickness 0.15)))
@@
         )
         (module W25Q128JVS (layer B.Cu)
-            (at 109.5375 42.862500000000004 90)
+            (at 109.5375 42.862500000000004 270)
             (fp_text reference "U2" (at 0 0 0) (layer "B.Fab")
               (effects (font (size 1 1) (thickness 0.15)))
@@
         )
         (module 1uF (layer B.Cu)
-            (at 116.475 42.862500000000004 90)
+            (at 104.77499999999999 42.862500000000004 270)
             (fp_text reference "C1" (at 0 0 0) (layer "B.Fab")
               (effects (font (size 1 1) (thickness 0.15)))
@@
         )
         (module 1uF (layer B.Cu)
-            (at 118.475 42.862500000000004 90)
+            (at 114.3 42.862500000000004 270)
             (fp_text reference "C2" (at 0 0 0) (layer "B.Fab")
               (effects (font (size 1 1) (thickness 0.15)))
@@
         )
         (module USBLC6-2SC6 (layer B.Cu)
-            (at 109.5375 47.862500000000004 90)
+            (at 119.0625 42.862500000000004 270)
             (fp_text reference "U3" (at 0 0 0) (layer "B.Fab")
               (effects (font (size 1 1) (thickness 0.15)))
@@
         )
         (module 10uF (layer B.Cu)
-            (at 142.875 47.62500000000001 90)
+            (at 138.35 47.62500000000001 90)
             (fp_text reference "C6" (at 0 0 0) (layer "B.Fab")
               (effects (font (size 1 1) (thickness 0.15)))
@@
         )
         (module 1uF (layer B.Cu)
-            (at 140.875 47.62500000000001 90)
+            (at 136.35 47.62500000000001 90)
             (fp_text reference "C7" (at 0 0 0) (layer "B.Fab")
               (effects (font (size 1 1) (thickness 0.15)))
@@
         )
         (module 100nF (layer B.Cu)
-            (at 138.875 47.62500000000001 90)
+            (at 134.35 47.62500000000001 90)
             (fp_text reference "C8" (at 0 0 0) (layer "B.Fab")
               (effects (font (size 1 1) (thickness 0.15)))
@@
         )
         (module 100nF (layer B.Cu)
-            (at 136.875 47.62500000000001 90)
+            (at 132.35 47.62500000000001 90)
             (fp_text reference "C9" (at 0 0 0) (layer "B.Fab")
               (effects (font (size 1 1) (thickness 0.15)))
@@
         )
         (module 100nF (layer B.Cu)
-            (at 134.875 47.62500000000001 90)
+            (at 130.35 47.62500000000001 90)
             (fp_text reference "C10" (at 0 0 0) (layer "B.Fab")
               (effects (font (size 1 1) (thickness 0.15)))
@@
         )
         (module 100nF (layer B.Cu)
-            (at 132.875 47.62500000000001 90)
+            (at 128.35 47.62500000000001 90)
             (fp_text reference "C11" (at 0 0 0) (layer "B.Fab")
               (effects (font (size 1 1) (thickness 0.15)))
@@
         )
         (module 100nF (layer B.Cu)
-            (at 136.875 52.3875 90)
+            (at 132.35 52.3875 90)
             (fp_text reference "C12" (at 0 0 0) (layer "B.Fab")
               (effects (font (size 1 1) (thickness 0.15)))
@@
         )
         (module 100nF (layer B.Cu)
-            (at 134.875 52.3875 90)
+            (at 130.35 52.3875 90)
             (fp_text reference "C13" (at 0 0 0) (layer "B.Fab")
               (effects (font (size 1 1) (thickness 0.15)))
@@
         )
         (module 100nF (layer B.Cu)
-            (at 132.875 52.3875 90)
+            (at 128.35 52.3875 90)
             (fp_text reference "C14" (at 0 0 0) (layer "B.Fab")
               (effects (font (size 1 1) (thickness 0.15)))
@@
         )
         (module 1uF (layer B.Cu)
-            (at 142.875 52.3875 90)
+            (at 138.35 52.3875 90)
             (fp_text reference "C15" (at 0 0 0) (layer "B.Fab")
               (effects (font (size 1 1) (thickness 0.15)))
@@
         )
         (module 100nF (layer B.Cu)
-            (at 140.875 52.3875 90)
+            (at 136.35 52.3875 90)
             (fp_text reference "C16" (at 0 0 0) (layer "B.Fab")
               (effects (font (size 1 1) (thickness 0.15)))
@@
         )
         (module 100nF (layer B.Cu)
-            (at 138.875 52.3875 90)
+            (at 134.35 52.3875 90)
             (fp_text reference "C17" (at 0 0 0) (layer "B.Fab")
               (effects (font (size 1 1) (thickness 0.15)))
